File: hardware/industrial-dual-0-20mA.kicad_pcb (KiCad board)
At the start: 2 copper layers, 40 x 40 mm, 38 parts, among them P1 CON-SENSOR2, P2 DEBUG, P3 BOOT, P4 P-PWR-8GN, Q1 FDN5630, U1 XMC1XXX24, U3 MCP3423, U4 DRILL, U5 DRILL, U6 DRILL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

Commit message: add two status leds, fix logo positions, fix text
Parts:
- removed R3: 1k, R0603F
- added D3: blue, kicad-libraries:D0603F, F.Cu at (126.3, 40.5)
- added D4: blue, kicad-libraries:D0603F, F.Cu at (127.9, 40.5)
- added RP2: 1k, kicad-libraries:4X0603, F.Cu at (105.4, 47.3)
- C1: footprint C0805 -> kicad-libraries:C0805
- C2, C4, C5, C6, FB1, FB2: footprint C0603 -> kicad-libraries:C0603
- C3: footprint C0402E -> kicad-libraries:C0402E
- C7, C8: footprint C0603F -> kicad-libraries:C0603F
- D1: footprint MiniMelf -> kicad-libraries:MiniMelf
- D2: footprint D0603F -> kicad-libraries:D0603F
- P1: footprint CON-SENSOR2 -> kicad-libraries:CON-SENSOR2
- P4: footprint OQ_8P -> kicad-libraries:OQ_8P
- Q1: footprint SOT23GDS -> kicad-libraries:SOT23GDS
- R1, R2, R4, R5, R8: footprint R0603 -> kicad-libraries:R0603
- R6, R7: footprint R0805 -> kicad-libraries:R0805
- RP1: footprint 4X0402 -> kicad-libraries:4X0402
- U3: footprint MSOP10-0.5 -> kicad-libraries:MSOP10-0.5
- U4, U5, U6, U7: footprint DRILL_NP -> kicad-libraries:DRILL_NP
- moved G*** 29.1 mm to (99.3, 59.7)
- moved G*** 26.1 mm to (127.8, 58.0), turned to 90 degrees
- moved VAL 19.0 mm to (117.8, 58.0), turned to 90 degrees
- moved VAL 18.8 mm to (107.8, 58.0), turned to 90 degrees
- moved P2 8.28 mm to (114.3, 51.1)
- moved P3 7.99 mm to (112.0, 52.6)
- moved D2 2.67 mm to (109.3, 40.6), turned to 270 degrees
Connections:
- P1 pad 1: Net-(P1-Pad1) -> (no net)
- U1 pad 11: Net-(U1-Pad11) -> (no net)
- U1 pad 13: Net-(P3-Pad2) -> Net-(RP2-Pad6)
- U1 pad 15: Net-(P2-Pad1) -> (no net)
- U1 pad 16: Net-(U1-Pad16) -> Net-(P3-Pad2)
- U1 pad 18: Net-(U1-Pad18) -> Net-(P2-Pad1)
- U1 pad 2: Net-(U1-Pad2) -> (no net)
- U1 pad 21: Net-(U1-Pad21) -> (no net)
- U1 pad 3: Net-(U1-Pad3) -> (no net)
- U1 pad 4: Net-(U1-Pad4) -> (no net)
- U1 pad 5: Net-(U1-Pad5) -> (no net)
- U1 pad 6: Net-(U1-Pad6) -> (no net)
- U1 pad 7: Net-(R3-Pad1) -> (no net)
- U1 pad 8: Net-(U1-Pad8) -> (no net)
- U3 pad 10: Net-(U3-Pad10) -> (no net)
Routing:
- net Net-(D4-Pad2): track 0.00 -> 24.9 mm
- net Net-(D3-Pad2): track 0.00 -> 23.7 mm
- net Net-(RP2-Pad8): track 0.00 -> 10.5 mm
- net GND: track 27.8 -> 37.5 mm
- net Net-(RP2-Pad6): track 0.00 -> 8.04 mm
- net 3V3: track 49.6 -> 57.5 mm, vias 2 -> 4
- net Net-(R3-Pad1): track 6.59 -> 0.00 mm
- net Net-(D2-Pad2): track 1.47 -> 8.03 mm
- net Net-(P2-Pad1): track 8.04 -> 1.78 mm
- net Net-(RP2-Pad5): track 0.00 -> 5.72 mm
- net Net-(P3-Pad2): track 8.27 -> 2.88 mm
Other:
- board text added: "0"
- board text added: "1"
