File: hardware/industrial-dual-0-20ma-v2.kicad_sch (KiCad schematic)
At the start: 35 parts, among them P1 CON-SENSOR2, P2 DEBUG, P3 BOOT, P4 P-PWR-8GN, Q1 FDN5630, U1 XMC1100, U3 MCP3423, U4 DRILL, U5 DRILL, U6 DRILL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

Commit message: Data Cleanup
Connections:
- net MEASURE is gone; now on net VCC: R2.1, R8.1
- net VCC: now reaches P4.1 (P1)
- net VCC: now also P4.3 (P3), P4.6 (P6)
Other:
- note added: "Copyright Tinkerforge GmbH 2023. This documentation describes Open Hardware and is licensed under the CERN OHL v. 1.1. You may redistribute and modify this documentation under the terms of the CERN OHL v.1.1. (http://ohwr.org/cernohl). This documentation is distributed WITHOUT ANY EXPRESS OR IMPLIED WARRANTY, INCLUDING OF MERCHANTABILITY, SATISFACTORY QUALITY AND FITNESS FOR A PARTICULAR PURPOSE.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"
- note removed: "Copyright Tinkerforge GmbH 2018. This documentation describes Open Hardware and is licensed under the CERN OHL v. 1.1. You may redistribute and modify this documentation under the terms of the CERN OHL v.1.1. (http://ohwr.org/cernohl). This documentation is distributed WITHOUT ANY EXPRESS OR IMPLIED WARRANTY, INCLUDING OF MERCHANTABILITY, SATISFACTORY QUALITY AND FITNESS FOR A PARTICULAR PURPOSE.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"
